File: pcb/bakeneko-60-pcb.kicad_pcb (KiCad board)
At the start: 2 copper layers, 284.7 x 94.2 mm, 154 parts, among them J1 JST SH 4-pin, J2 AVR-ISP-6, SW1 Reset, U1 SRV05-4, U2 ATmega32U4-AU, Y1 16MHz

Commit message: remove 6.25u bottom row
Parts:
- removed MX59, MX60, MX61, MX64, MX65, MX66: 1.25u, MX_Only:MXOnly-1.25U-NoLED
- removed MX62: 6.25u, MX_Only:MXOnly-6.25U-ReversedStabilizers-NoLED
Connections:
- U1 pad 3: Net-(U1-Pad3) -> unconnected-(U1-Pad3)
- U1 pad 4: Net-(U1-Pad4) -> unconnected-(U1-Pad4)
- U2 pad 18: Net-(U2-Pad18) -> unconnected-(U2-Pad18)
- U2 pad 41: Net-(U2-Pad41) -> unconnected-(U2-Pad41)
- U2 pad 42: Net-(U2-Pad42) -> unconnected-(U2-Pad42)
Routing:
- net COL2: track 145.1 -> 142.7 mm
- net Net-(D63-Pad2): track 9.25 -> 6.87 mm
- net Net-(D56-Pad2): track 15.4 -> 13.0 mm
- net Net-(D61-Pad2): track 9.20 -> 6.82 mm
- net COL1: track 110.2 -> 107.8 mm
- net COL0: track 100.5 -> 98.1 mm
- net Net-(D62-Pad2): track 9.25 -> 6.87 mm
Other:
- outline, holes or cut-outs redrawn
- net class D removed
- net class Default removed
- net class Power removed
