File: pcb/bakeneko-60-pcb.kicad_pcb (KiCad board)
At the start: 2 copper layers, 284.7 x 94.2 mm, 151 parts, among them J1 JST SH 4-pin, J2 AVR-ISP-6, SW1 Reset, U1 SRV05-4, U2 ATmega32U4-AU, Y1 16MHz

Commit message: no corner outline
Parts:
- added G***: LOGO, bakeneko:outline_no_corner, F.Cu at (141.4, 47.0)
Other:
- board size 284.7 x 94.2 mm -> 284.8 x 106.7 mm

Commit message: remove silk overlay placeholder
Parts:
- removed G***: LOGO, bakeneko:outline_no_corner

Commit message: move text to center
Other:
- board text added: "40-ish by InternetbaroN v1.0"
- board text removed: "40-ish by InternetbaroN"
Changed lines of the file:
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@@
       (xy 59.693314 -6.382929)
     ) (layer "Edge.Cuts") (width 0.2) (fill none))
-  (gr_text "40-ish by InternetbaroN" (at 274.915477 91.907501) (layer "B.SilkS")
+  (gr_text "40-ish by InternetbaroN v1.0" (at 143.46 56.63) (layer "B.SilkS")
     (effects (font (size 1 1) (thickness 0.15)) (justify mirror))
   )
