File: pcb/matrix.kicad_sch (KiCad schematic)
At the start: 133 parts

Commit message: generic layout baseline
Parts:
- added MX80: 7u-10u, MX_Only:MXOnly-10U-7U-ReversedStabilizers-NoLED, symbol Switch:SW_SPST
- MX63, MX74: value 1.25u -> 1u; footprint MX_Only:MXOnly-1.25U-NoLED -> MX_Only:MXOnly-1U-NoLED
- MX69: value 1.25u -> 1.5u; footprint MX_Only:MXOnly-1.25U-NoLED -> MX_Only:MXOnly-1.5U-NoLED
- MX70: value 2.75u -> 2.25u; footprint MX_Only:MXOnly-2.75U-ReversedStabilizers-NoLED -> MX_Only:MXOnly-2.25U-ReversedStabilizers-NoLED
- MX75: value 2u -> 2.75u; footprint MX_Only:MXOnly-2U-ReversedStabilizers-NoLED -> MX_Only:MXOnly-2.75U-ReversedStabilizers-NoLED
Connections:
- net COL6: now also MX80.2 (B)
- net at D59.2 (A), MX70.1 (A): now also MX80.1 (A)
Changed lines of the file:
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@@
   (junction (at 181.61 100.33) (diameter 0) (color 0 0 0 0)
   )
+  (junction (at 142.24 129.54) (diameter 0) (color 0 0 0 0)
+  )
   (junction (at 59.69 74.93) (diameter 0) (color 0 0 0 0)
   )
@@
   (junction (at 171.45 39.37) (diameter 0) (color 0 0 0 0)
   )
+  (junction (at 129.54 129.54) (diameter 0) (color 0 0 0 0)
+  )
   (junction (at 227.33 92.71) (diameter 0) (color 0 0 0 0)
   )
@@
     (stroke (width 0) (type default) (color 0 0 0 0))
   )
+  (wire (pts (xy 142.24 142.24) (xy 142.24 129.54))
+    (stroke (width 0) (type default) (color 0 0 0 0))
+  )
   (wire (pts (xy 101.6 39.37) (xy 101.6 57.15))
     (stroke (width 0) (type default) (color 0 0 0 0))
@@
     (stroke (width 0) (type default) (color 0 0 0 0))
   )
+  (wire (pts (xy 129.54 129.54) (xy 129.54 142.24))
+    (stroke (width 0) (type default) (color 0 0 0 0))
+  )
   (wire (pts (xy 111.76 64.77) (xy 125.73 64.77))
     (stroke (width 0) (type default) (color 0 0 0 0))
@@
     (stroke (width 0) (type default) (color 0 0 0 0))
   )
+  (wire (pts (xy 129.54 142.24) (xy 130.81 142.24))
+    (stroke (width 0) (type default) (color 0 0 0 0))
+  )
   (wire (pts (xy 129.54 74.93) (xy 129.54 92.71))
     (stroke (width 0) (type default) (color 0 0 0 0))
@@
     (stroke (width 0) (type default) (color 0 0 0 0))
   )
+  (wire (pts (xy 140.97 142.24) (xy 142.24 142.24))
+    (stroke (width 0) (type default) (color 0 0 0 0))
+  )
   (wire (pts (xy 251.46 30.48) (xy 251.46 39.37))
     (stroke (width 0) (type default) (color 0 0 0 0))
@@
     (in_bom yes) (on_board yes)
     (property "Reference" "MX70" (id 0) (at 134.62 123.571 0))
-    (property "Value" "2.75u" (id 1) (at 134.62 125.8824 0))
-    (property "Footprint" "MX_Only:MXOnly-2.75U-ReversedStabilizers-NoLED" (id 2) (at 134.62 129.54 0)
+    (property "Value" "2.25u" (id 1) (at 134.62 125.8824 0))
+    (property "Footprint" "MX_Only:MXOnly-2.25U-ReversedStabilizers-NoLED" (id 2) (at 134.62 129.54 0)
       (effects (font (size 1.27 1.27)) hide)
     )
@@
     (in_bom yes) (on_board yes)
     (property "Reference" "MX69" (id 0) (at 78.74 123.571 0))
-    (property "Value" "1.25u" (id 1) (at 78.74 125.8824 0))
-    (property "Footprint" "MX_Only:MXOnly-1.25U-NoLED" (id 2) (at 78.74 129.54 0)
+    (property "Value" "1.5u" (id 1) (at 78.74 125.8824 0))
+    (property "Footprint" "MX_Only:MXOnly-1.5U-NoLED" (id 2) (at 78.74 129.54 0)
       (effects (font (size 1.27 1.27)) hide)
     )
@@
     (in_bom yes) (on_board yes)
     (property "Reference" "MX63" (id 0) (at 190.5 104.521 0))
-    (property "Value" "1.25u" (id 1) (at 190.5 106.8324 0))
-    (property "Footprint" "MX_Only:MXOnly-1.25U-NoLED" (id 2) (at 190.5 110.49 0)
+    (property "Value" "1u" (id 1) (at 190.5 106.8324 0))
+    (property "Footprint" "MX_Only:MXOnly-1U-NoLED" (id 2) (at 190.5 110.49 0)
       (effects (font (size 1.27 1.27)) hide)
     )
@@
     (in_bom yes) (on_board yes)
     (property "Reference" "MX74" (id 0) (at 106.68 123.571 0))
-    (property "Value" "1.25u" (id 1) (at 106.68 125.8824 0))
-    (property "Footprint" "MX_Only:MXOnly-1.25U-NoLED" (id 2) (at 106.68 129.54 0)
+    (property "Value" "1u" (id 1) (at 106.68 125.8824 0))
+    (property "Footprint" "MX_Only:MXOnly-1U-NoLED" (id 2) (at 106.68 129.54 0)
       (effects (font (size 1.27 1.27)) hide)
     )
@@
     (pin "2")
   )
+  (symbol (lib_id "Switch:SW_SPST") (at 135.89 142.24 0) (mirror y) (unit 1)
+    (in_bom yes) (on_board yes)
+    (property "Reference" "MX80" (id 0) (at 135.89 136.271 0))
+    (property "Value" "7u-10u" (id 1) (at 135.89 138.5824 0))
+    (property "Footprint" "MX_Only:MXOnly-10U-7U-ReversedStabilizers-NoLED" (id 2) (at 135.89 142.24 0)
+      (effects (font (size 1.27 1.27)) hide)
+    )
+    (property "Datasheet" "~" (id 3) (at 135.89 142.24 0)
+      (effects (font (size 1.27 1.27)) hide)
+    )
+    (pin "1")
+    (pin "2")
+  )
   (symbol (lib_id "Switch:SW_SPST") (at 167.64 129.54 0) (mirror y) (unit 1)
     (in_bom yes) (on_board yes)
     (property "Reference" "MX75" (id 0) (at 167.64 123.571 0))
-    (property "Value" "2u" (id 1) (at 167.64 125.8824 0))
-    (property "Footprint" "MX_Only:MXOnly-2U-ReversedStabilizers-NoLED" (id 2) (at 167.64 129.54 0)
+    (property "Value" "2.75u" (id 1) (at 167.64 125.8824 0))
+    (property "Footprint" "MX_Only:MXOnly-2.75U-ReversedStabilizers-NoLED" (id 2) (at 167.64 129.54 0)
       (effects (font (size 1.27 1.27)) hide)
     )
